File: PCB/Ouidire_v1/Ouidire_v1.kicad_pcb (KiCad board)
At the start: 2 copper layers, 12 parts, among them J1 Conn_01x01_Female

Commit message: pcb v1 ok
Parts:
- removed J1: Conn_01x01_Female, Connector_PinSocket_2.54mm:PinSocket_1x01_P2.54mm_Vertical
- added VUSB+: Conn_01x01_Female, Connector_PinSocket_2.54mm:PinSocket_1x01_P2.54mm_Vertical, F.Cu at (154.9, 116.8)
- moved R2 16.0 mm to (150.1, 78.2), turned to 90 degrees
- moved JST_LedBtn1 15.9 mm to (148.6, 112.3), turned to 180 degrees
- moved R1 14.5 mm to (150.1, 84.5), turned to 90 degrees
- moved R3 8.64 mm to (151.8, 109.2), turned to 90 degrees
- moved Coil2 5.24 mm to (153.7, 127.0), turned to 270 degrees
Connections:
- TTGO_T8_V1.7_R1 pad 12: Net-(TTGO_T8_V1.7_R1-Pad12) -> GND
Routing:
- net +3V3: track 0.00 -> 57.0 mm
- net Net-(J1-Pad1): track 0.00 -> 38.6 mm, vias 0 -> 1
- net RX: track 0.00 -> 36.7 mm, vias 0 -> 1
- net TX: track 0.00 -> 35.3 mm
- net BCK: track 0.00 -> 35.3 mm
- net LCK: track 0.00 -> 33.9 mm, vias 0 -> 1
- net RST: track 0.00 -> 30.5 mm
- net Net-(Coil1-Pad1): track 0.00 -> 17.9 mm
- net Net-(Coil1-Pad2): track 0.00 -> 12.0 mm
- net DOUT: track 0.00 -> 10.8 mm
- net Net-(R1-Pad2): track 0.00 -> 8.81 mm
- net GND: track 0.00 -> 7.98 mm
- net LED: track 0.00 -> 6.37 mm
- net Net-(JST_LedBtn1-Pad3): track 0.00 -> 3.40 mm
- added copper zone on F.Cu, net GND
Other:
- board outline added: 32.5 x 59.2 mm
- board text added: "100kΩ"
- board text added: "4kΩ"
- board text added: "Btn+"
- board text added: "Btn-"
- board text added: "COIL"
- board text added: "Led+"
- board text added: "Led-"
- board text added: "Ouidire_v1_Hemisphere_10.2022"
- board text added: "TVS"
