File: PCB/Ouidire_v1/Ouidire_v1.sch (KiCad schematic (older format))
At the start: 12 parts, among them J1 Conn_01x01_Female

Commit message: pcb v1 ok
Connections:
- net GND: now also TTGO_T8_V1.7_R1.12 (Pin_12)
Changed lines of the file:
@@
 Text Notes 5000 3650 0    50   ~ 0
 VIN
+$Comp
+L power:GND #PWR?
+U 1 1 633C022B
+P 3400 2750
+F 0 "#PWR?" H 3400 2500 50  0001 C CNN
+F 1 "GND" V 3405 2622 50  0000 R CNN
+F 2 "" H 3400 2750 50  0001 C CNN
+F 3 "" H 3400 2750 50  0001 C CNN
+	1    3400 2750
+	0    1    1    0
+$EndComp
 $EndSCHEMATC
